Commit message: Added all the necessary Files for Sim

File: husky_ur_description/urdf/husky_ur5_description.urdf.xacro (robot description, xacro)
@@ -5,5 +5,5 @@
     <parent link="top_plate_front_link" />
     <child link="ur_arm_base_link" />
-    <origin xyz="$(optenv HUSKY_UR_XYZ -0.105 0.0 0.0)" rpy="$(optenv HUSKY_UR_RPY 0 0 3.1415927)"/>
+    <origin xyz="$(optenv HUSKY_UR_XYZ -0.4 0.0 0.0)" rpy="$(optenv HUSKY_UR_RPY 0 0 3.1415927)"/>
   </joint>
   <xacro:ur5_robot prefix="ur_arm_" joint_limited="true"/>
