Commit message: Fixed Arm issue in MoveIt

File: husky/husky_description/urdf/accessories/sick_lms1xx_mount.urdf.xacro (robot description, xacro)
@@ -36,10 +36,10 @@
         </geometry>
       </visual>
-      <collision>
+      <!-- <collision>
         <origin xyz="0 0 .0585" rpy="0 0 0" />
         <geometry>
           <box size=".1 .108 .117" />
         </geometry>
-      </collision>
+      </collision> -->
     </link>
     <joint name="${prefix}_laser_joint" type="fixed">

File: husky_ur_description/urdf/husky_ur5_description.urdf.xacro (robot description, xacro)
@@ -5,5 +5,5 @@
     <parent link="top_plate_front_link" />
     <child link="ur_arm_base_link" />
-    <origin xyz="$(optenv HUSKY_UR_XYZ -0.4 0.0 0.0)" rpy="$(optenv HUSKY_UR_RPY 0 0 3.1415927)"/>
+    <origin xyz="$(optenv HUSKY_UR_XYZ -0.45 0.0 0.0)" rpy="$(optenv HUSKY_UR_RPY 0 0 3.1415927)"/>
   </joint>
   <xacro:ur5_robot prefix="ur_arm_" joint_limited="true"/>
